File: Kai_car/Kai_car.kicad_sch (KiCad schematic)
At the start: 16 parts, among them M1 Motor_DC, M2 Motor_DC

Commit message: checkpoint_2
Parts:
- removed BT1: 6V, symbol Device:Battery
- removed D3: White_1, symbol Device:LED
- removed D4: white_2, symbol Device:LED
- added C3: 0.1u, symbol Device:C
- added C4: 470u, symbol Device:C
- added C5: 0.01, symbol Device:C
- added C6: 100u, symbol Device:C
- added D1: White_2, symbol Device:LED
- added D2: White_1, symbol Device:LED
- added D7: 1N4007, Diode_THT:D_DO-41_SOD81_P10.16mm_Horizontal, symbol Diode:1N4007
- added J1, J2: Conn_01x02_Pin, symbol Connector:Conn_01x02_Pin
- added J3: Conn_01x04_Pin, symbol Connector:Conn_01x04_Pin
- added Q1, Q2: BC547, Package_TO_SOT_THT:TO-92_Inline, symbol Transistor_BJT:BC547
- added R10, R7, R8, R9: 10k, symbol Device:R_US
- added R11: 50, symbol Device:R
- added R12: 100k, symbol Device:R
- added R13, R14, R15, R5, R6: 10k, symbol Device:R
- added TP1: VCC, symbol Connector:TestPoint
- added TP2, TP5: GND, symbol Connector:TestPoint
- added TP3, TP6: 3V3, symbol Connector:TestPoint
- added TP4: DAC, symbol Connector:TestPoint
- added U2: ~, symbol Custom_Symbols:oled_screen_kai
- added U3: LM386, symbol Amplifier_Audio:LM386
- added U4: PCM5102A, Package_SO:TSSOP-20_4.4x6.5mm_P0.65mm, symbol Audio:PCM5102A
- C2: value 10u -> 470u
- LS1: value Piezo_Buzzer -> 4ohm_spk
- R1, R2: value 85 -> 200
- R3, R4: value 65 -> 200
Connections:
- net GND: now also U1.14 (GND), U1.29 (GND), C6.2, J2.2 (Pin_2), J3.3 (Pin_3), Q1.3 (E), Q2.3 (E), R10.2, R11.2, R13.2, R6.2, R7.2, R8.2, R9.2, U2. (SDA), U3.2 (-), U3.4 (GND), U4.12 (SCK), U4.19 (DGND), U4.3 (CPGND), U4.9 (AGND); no longer R1.2, R2.2
- net LM_A: now also R8.1
- net LM_B: now also R7.1
- net RM_A: now also R10.1
- net RM_B: now also R9.1
- net SCL: now also J3.2 (Pin_2), U2. (SDA)
- net SDA: now also J3.1 (Pin_1), U2. (SDA)
- net VCC: now also R1.1, R2.1, U1.15 (VIN), C6.1, D7.1 (K), R5.1, U3.6 (V+)
- net back_lights: now also D5.2 (A), D6.2 (A), U1.11 (D14); no longer D5.1 (K), D6.1 (K)
- net front_lights: now also U1.13 (D13), R14.1, R15.1
- net DIN: now reaches U1.21 (D19)
- net DIN: now also U4.14 (DIN)
- net LRCK: now reaches U1.22 (D18)
- net LRCK: now also U4.15 (LRCK)
- net BCK: now reaches U1.23 (D5)
- net BCK: now also U4.13 (BCK)
- net 3V3: now reaches U1.30 (3v3)
- net 3V3: now also DRV1.1 (EEP), J3.4 (Pin_4), U2. (SDA), U4.1 (CPVDD), U4.20 (DVDD), U4.8 (AVDD)
- net ADC: now reaches U1.4 (D34)
- net ADC: now also R5.2, R6.1
- net at R3.1: now also D5.1 (K); no longer D5.2 (A)
- net at R4.1: now also D6.1 (K); no longer D6.2 (A)
- net speaker: no longer names the net of LS1.1
- net speaker: now also C4.2
- new net: C3.2, U3.3 (+)
- new net: C4.1, C5.1, U3.5
- new net: C3.1, R12.2, R13.1
- new net: D2.1 (K), Q2.1 (C)
- new net: D2.2 (A), R1.2
- new net: Q1.2 (B), R14.2
- new net: D1.1 (K), Q1.1 (C)
- new net: D1.2 (A), R2.2
- new net: Q2.2 (B), R15.2
- new net: C5.2, R11.1
- new net Batt_1+: D7.2 (A), J1.1 (Pin_1)
- new net Batt_1-: J1.2 (Pin_2)
- new net Batt_2+: J2.1 (Pin_1)
- new net DAC: R12.1, U4.6 (OUTL)
- no-connect marks 0 -> 24
Other:
- note added: "1. Find Diode to prevent Back-voltage 2. Plug in Front and Back LEDs with corresponding resistors 3. Find high power diode to prevent reverse Polarity damage 4. Configure an alert if batteries plugged in backwards"
- note added: "Battery Indicator"
- note added: "TODO"
- moved on the sheet: C1, C2, D5, D6, LS1, R3, R4, U1
