File: Kai_car/_autosave-Kai_car.kicad_sch (KiCad schematic)
At the start: 21 parts, among them M1 Motor_DC, M2 Motor_DC

Commit message: checkpoint_2
Parts:
- removed BT1: 6V, symbol Device:Battery
- removed D1, D2: 1N4007, Diode_THT:D_DO-41_SOD81_P10.16mm_Horizontal, symbol Diode:1N4007
- removed D3: White_1, symbol Device:LED
- removed D4: white_2, symbol Device:LED
- added C3: 0.1u, symbol Device:C
- added C4: 100u, symbol Device:C
- added C5: 0.01, symbol Device:C
- added C6: 470u, symbol Device:C
- added D1: White_2, symbol Device:LED
- added D2: White_1, symbol Device:LED
- added D7: 1N4007, Diode_THT:D_DO-41_SOD81_P10.16mm_Horizontal, symbol Diode:1N4007
- added J1, J2: Conn_01x02_Pin, symbol Connector:Conn_01x02_Pin
- added J3: Conn_01x04_Pin, symbol Connector:Conn_01x04_Pin
- added Q1, Q2: BC547, Package_TO_SOT_THT:TO-92_Inline, symbol Transistor_BJT:BC547
- added R10, R7, R8, R9: 10k, symbol Device:R_US
- added R11: 50, symbol Device:R
- added R12, R14, R15: 10k, symbol Device:R
- added R13: 100, symbol Device:R
- added TP1: VCC, symbol Connector:TestPoint
- added TP2, TP5: GND, symbol Connector:TestPoint
- added TP3, TP6: 3V3, symbol Connector:TestPoint
- added TP4: DAC, symbol Connector:TestPoint
- added U3: LM386, symbol Amplifier_Audio:LM386
- added U4: PCM5102A, Package_SO:TSSOP-20_4.4x6.5mm_P0.65mm, symbol Audio:PCM5102A
- C2: value 10u -> 470u
- LS1: value Piezo_Buzzer -> 4ohm_spk
- R1, R2: value 85 -> 200
- R3, R4: value 65 -> 200
Connections:
- net 3V3: now also DRV1.1 (EEP), J3.4 (Pin_4), U4.1 (CPVDD), U4.20 (DVDD), U4.8 (AVDD)
- net GND: now also C6.2, J2.2 (Pin_2), J3.3 (Pin_3), Q1.3 (E), Q2.3 (E), R10.2, R11.2, R13.2, R7.2, R8.2, R9.2, U3.2 (-), U3.4 (GND), U4.12 (SCK), U4.19 (DGND), U4.3 (CPGND), U4.9 (AGND); no longer R1.2, R2.2
- net LM_A: now also DRV1.7 (In4), U1.10 (D27), R7.1; no longer DRV1.8 (In3), U1.8 (D25)
- net LM_B: now also DRV1.8 (In3), U1.9 (D26), R8.1; no longer DRV1.7 (In4), U1.7 (D33)
- net RM_A: now also U1.23 (D5), R10.1; no longer U1.10 (D27)
- net RM_B: now also U1.22 (D18), R9.1; no longer U1.9 (D26)
- net SCL: now also J3.2 (Pin_2)
- net SDA: now also J3.1 (Pin_1)
- net VCC: now also R1.1, R2.1, U1.15 (VIN), C6.1, D7.1 (K), U3.6 (V+)
- net back_lights: now also D5.2 (A), D6.2 (A); no longer D5.1 (K), D6.1 (K)
- net front_lights: now also R14.1, R15.1
- net at R3.1: now also D5.1 (K); no longer D5.2 (A)
- net at R4.1: now also D6.1 (K); no longer D6.2 (A)
- net speaker: no longer names the net of LS1.1
- net speaker: now also C4.2; no longer U1.16 (D23)
- new net: C3.2, U3.3 (+)
- new net: C4.1, C5.1, U3.5
- new net: C3.1, R12.2, R13.1
- new net: D2.1 (K), Q2.1 (C)
- new net: D2.2 (A), R1.2
- new net: Q1.2 (B), R14.2
- new net: D1.1 (K), Q1.1 (C)
- new net: D1.2 (A), R2.2
- new net: Q2.2 (B), R15.2
- new net: C5.2, R11.1
- new net BCK: U4.13 (BCK)
- new net Batt_1+: D7.2 (A), J1.1 (Pin_1)
- new net Batt_1-: J1.2 (Pin_2)
- new net Batt_2+: J2.1 (Pin_1)
- new net DAC: R12.1, U4.6 (OUTL)
- new net DIN: U4.14 (DIN)
- new net LRCK: U4.15 (LRCK)
- no-connect marks 18 -> 29
Other:
- note removed: "1. Find Diode to prevent Back-voltage 2. Plug in Front and Back LEDs with corresponding resistors 3. Find high power diode to prevent reverse Polarity damage 4. Configure an alert if batteries plugged in backwards"
- note removed: "TODO"
- moved on the sheet: C1, C2, D5, D6, LS1, R3, R4, U1, U2
